File: kr556rt2.kicad_sch (KiCad schematic)
At the start: 2 parts, among them U1 27C512, U2 КР556РТ2

Commit message: Update 22.07.2023 - Gerbers ver1
Parts:
- added U3: КР556РТ2, Package_DIP:DIP-28_W15.24mm_Socket, symbol kr556rt2_eprom:КР556РТ2
- added U4: 27C512, Package_DIP:DIP-28_W15.24mm, symbol Memory_EPROM:27C512
Connections:
- new net: U3.20 (А16), U4.1 (A15)
- new net: U3.9 (А1), U4.10 (A0)
- new net: U3.18 (В1), U4.11 (D0)
- new net: U3.17 (В2), U4.12 (D1)
- new net: U3.16 (В3), U4.13 (D2)
- new net: U3.14 (GND), U4.14 (GND)
- new net: U3.15 (В4), U4.15 (D3)
- new net: U3.13 (В5), U4.16 (D4)
- new net: U3.12 (В6), U4.17 (D5)
- new net: U3.11 (В7), U4.18 (D6)
- new net: U3.10 (В8), U4.19 (D7)
- new net: U3.23 (А13), U4.2 (A12)
- new net: U3.19 (РВ), U4.20 (~{CE})
- new net: U3.25 (А11), U4.21 (A10)
- new net: U3.24 (А12), U4.23 (A11)
- new net: U3.26 (А10), U4.24 (A9)
- new net: U3.27 (А9), U4.25 (A8)
- new net: U3.22 (А14), U4.26 (A13)
- new net: U3.21 (А15), U4.27 (A14)
- new net: U3.28 (Vcc), U4.28 (VCC)
- new net: U3.2 (А8), U4.3 (A7)
- new net: U3.3 (А7), U4.4 (A6)
- new net: U3.4 (А6), U4.5 (A5)
- new net: U3.5 (А5), U4.6 (A4)
- new net: U3.6 (А4), U4.7 (A3)
- new net: U3.7 (А3), U4.8 (A2)
- new net: U3.8 (А2), U4.9 (A1)
- no-connect marks 1 -> 2
