File: kr556rt2.kicad_pcb (KiCad board)
At the start: 2 copper layers, 24.8 x 40.1 mm, 2 parts, among them U1 27C512, U2 КР556РТ2

Commit message: Update kr556rt2.kicad_pcb
Parts:
- moved U2 1.05 mm to (66.7, 41.8)
- moved U1 0.05 mm to (62.8, 41.8)
Routing:
- net Net-(U1-A13): track 15.5 -> 12.1 mm
- net Net-(U1-A10): track 11.7 -> 13.8 mm
- net Net-(U1-VCC): track 2.85 -> 3.90 mm
- net Net-(U1-D3): track 2.85 -> 3.90 mm
- net Net-(U1-GND): track 2.85 -> 3.90 mm
- net Net-(U1-D0): track 19.1 -> 20.1 mm
- net Net-(U1-D2): track 19.1 -> 20.1 mm
- net Net-(U1-D1): track 19.1 -> 20.1 mm
- net Net-(U1-D7): track 12.4 -> 11.4 mm
- net Net-(U1-D5): track 12.4 -> 11.4 mm
- net Net-(U1-D6): track 12.4 -> 11.4 mm
- net Net-(U1-D4): track 12.4 -> 11.4 mm
- net Net-(U1-~{CE}): track 4.54 -> 5.51 mm
- net Net-(U1-A15): track 31.8 -> 30.9 mm
- net Net-(U1-A11): track 4.56 -> 5.43 mm
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Other:
- board size 24.8 x 40.1 mm -> 23.5 x 39.4 mm

Commit message: Update 22.07.2023 - Gerbers ver1
Parts:
- added U3: КР556РТ2, convertor_kr:DIP-28_W15.24mm_Socket, F.Cu at (89.4, 41.1)
- added U4: 27C512, convertor_kr:DIP-28_W15.24mm, F.Cu at (93.4, 41.1)
- added mouse-bite-2.54mm-slot_13: VAL**, convertor_kr:mouse-bite-2.54mm-slot, F.Cu at (85.0, 71.7)
- added mouse-bite-2.54mm-slot_13: VAL**, convertor_kr:mouse-bite-2.54mm-slot, F.Cu at (85.0, 69.4)
- added mouse-bite-2.54mm-slot_13: VAL**, convertor_kr:mouse-bite-2.54mm-slot, F.Cu at (85.0, 59.2)
- added mouse-bite-2.54mm-slot_13: VAL**, convertor_kr:mouse-bite-2.54mm-slot, F.Cu at (85.0, 46.7)
- added mouse-bite-2.54mm-slot_13: VAL**, convertor_kr:mouse-bite-2.54mm-slot, F.Cu at (85.0, 56.9)
- added mouse-bite-2.54mm-slot_13: VAL**, convertor_kr:mouse-bite-2.54mm-slot, F.Cu at (85.0, 44.4)
- U1: footprint Package_DIP:DIP-28_W15.24mm -> convertor_kr:DIP-28_W15.24mm
- U2: footprint Package_DIP:DIP-28_W15.24mm_Socket -> convertor_kr:DIP-28_W15.24mm_Socket
- moved U2 1.53 mm to (65.3, 41.1)
- moved U1 1.53 mm to (61.4, 41.1)
Routing:
- net Net-(U3-А16): track 0.00 -> 25.6 mm
- net Net-(U3-А15): track 0.00 -> 22.5 mm
- net Net-(U3-В8): track 0.00 -> 20.2 mm
- net Net-(U3-В7): track 0.00 -> 20.2 mm
- net Net-(U3-В6): track 0.00 -> 20.2 mm
- net Net-(U3-В5): track 0.00 -> 20.2 mm
- net Net-(U3-А11): track 0.00 -> 15.5 mm
- net Net-(U3-А13): track 0.00 -> 15.4 mm
- net Net-(U3-А14): track 0.00 -> 11.8 mm
- net Net-(U3-В3): track 0.00 -> 11.2 mm
- net Net-(U3-В2): track 0.00 -> 11.2 mm
- net Net-(U3-В1): track 0.00 -> 11.2 mm
- net Net-(U3-А9): track 0.00 -> 6.75 mm
- net Net-(U3-А10): track 0.00 -> 6.75 mm
- net Net-(U3-А2): track 0.00 -> 5.09 mm
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Other:
- board size 23.5 x 39.4 mm -> 52.9 x 40 mm
- board text added: "MadCat 2023 Ver.1"
- board text added: "Read КР556РТ2 as 27C512"
- board text added: "Top"
- board text added: "Use 27C512 as КР556РТ2"
- board text added: "https://github.com/madcatse/DeltaS-KR556RT2-EPROM"
- board text added: "https://t.me/zx_delta_s"

Commit message: Update kr556rt2.kicad_pcb
Other:
- board size 52.9 x 40 mm -> 52.9 x 38.7 mm
Changed lines of the file:
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@@
         (effects (font (size 1 1) (thickness 0.15)))
     )
-    (fp_text value "27C512" (at 7.0612 35.4076) (layer "F.SilkS")
+    (fp_text value "27C512" (at 6.133307 35.86195) (layer "F.SilkS")
         (effects (font (size 1 1) (thickness 0.15)))
     )
@@
         (effects (font (size 1 1) (thickness 0.15)))
     )
-    (fp_text value "КР556РТ2" (at 7.0104 35.38345) (layer "F.SilkS")
+    (fp_text value "КР556РТ2" (at 5.588 35.56125) (layer "F.SilkS")
         (effects (font (size 1 1) (thickness 0.15)))
     )
@@
   (gr_circle (center 87.1474 41.1734) (end 87.57014 41.1734)
     (stroke (width 0.2) (type solid)) (fill solid) (layer "F.SilkS"))
-  (gr_line (start 59.547 38.1) (end 82.560123 38.1)
+  (gr_line (start 59.547 39.4) (end 82.560123 39.4)
     (stroke (width 0.1) (type default)) (layer "Edge.Cuts"))
   (gr_arc (start 83.560123 74.321277) (mid 84.9884 72.893) (end 86.416677 74.321277)
@@
   (gr_line (start 87.416677 78.1) (end 110.4298 78.1)
     (stroke (width 0.1) (type default)) (layer "Edge.Cuts"))
-  (gr_arc (start 86.416677 39.1) (mid 86.70957 38.392893) (end 87.416677 38.1)
-    (stroke (width 0.1) (type default)) (layer "Edge.Cuts"))
-  (gr_arc (start 110.4298 38.1) (mid 111.136907 38.392893) (end 111.4298 39.1)
+  (gr_arc (start 86.416677 40.4) (mid 86.709569 39.692885) (end 87.416677 39.4)
+    (stroke (width 0.1) (type default)) (layer "Edge.Cuts"))
+  (gr_arc (start 110.4298 39.4) (mid 111.136907 39.692893) (end 111.4298 40.4)
     (stroke (width 0.1) (type default)) (layer "Edge.Cuts"))
   (gr_line (start 83.566 66.907484) (end 83.566 61.6966)
@@
   (gr_arc (start 87.416677 78.1) (mid 86.709585 77.807099) (end 86.416677 77.1)
     (stroke (width 0.1) (type default)) (layer "Edge.Cuts"))
-  (gr_line (start 87.416677 38.1) (end 110.4298 38.1)
-    (stroke (width 0.1) (type default)) (layer "Edge.Cuts"))
-  (gr_arc (start 82.560123 38.1) (mid 83.26723 38.392893) (end 83.560123 39.1)
+  (gr_line (start 87.416677 39.4) (end 110.4298 39.4)
+    (stroke (width 0.1) (type default)) (layer "Edge.Cuts"))
+  (gr_arc (start 82.560123 39.4) (mid 83.267215 39.692901) (end 83.560123 40.4)
     (stroke (width 0.1) (type default)) (layer "Edge.Cuts"))
   (gr_arc (start 83.566 61.6966) (mid 84.994277 60.268323) (end 86.422554 61.6966)
@@
   (gr_arc (start 59.547 78.1) (mid 58.839893 77.807107) (end 58.547 77.1)
     (stroke (width 0.1) (type default)) (layer "Edge.Cuts"))
-  (gr_line (start 58.547 39.1) (end 58.547 77.1)
+  (gr_line (start 58.547 40.4) (end 58.547 77.1)
     (stroke (width 0.1) (type default)) (layer "Edge.Cuts"))
   (gr_arc (start 83.566 49.231077) (mid 84.994277 47.8028) (end 86.422554 49.231077)
@@
   (gr_line (start 86.416677 74.321277) (end 86.416677 77.1)
     (stroke (width 0.1) (type default)) (layer "Edge.Cuts"))
-  (gr_arc (start 58.547 39.1) (mid 58.839893 38.392893) (end 59.547 38.1)
-    (stroke (width 0.1) (type default)) (layer "Edge.Cuts"))
-  (gr_line (start 83.560123 41.878723) (end 83.560123 39.1)
+  (gr_arc (start 58.547 40.4) (mid 58.839893 39.692893) (end 59.547 39.4)
+    (stroke (width 0.1) (type default)) (layer "Edge.Cuts"))
+  (gr_line (start 83.560123 41.878723) (end 83.560123 40.4)
     (stroke (width 0.1) (type default)) (layer "Edge.Cuts"))
   (gr_line (start 86.422554 54.441961) (end 86.422554 49.231077)
     (stroke (width 0.1) (type solid)) (layer "Edge.Cuts"))
-  (gr_line (start 111.4298 39.1) (end 111.4298 77.1)
+  (gr_line (start 111.4298 40.4) (end 111.4298 77.1)
     (stroke (width 0.1) (type default)) (layer "Edge.Cuts"))
   (gr_arc (start 111.4298 77.1) (mid 111.136907 77.807107) (end 110.4298 78.1)
@@
   (gr_arc (start 86.422554 54.441961) (mid 84.994277 55.870238) (end 83.566 54.441961)
     (stroke (width 0.1) (type solid)) (layer "Edge.Cuts"))
-  (gr_line (start 86.416677 41.878723) (end 86.416677 39.1)
+  (gr_line (start 86.416677 41.878723) (end 86.416677 40.4)
     (stroke (width 0.1) (type default)) (layer "Edge.Cuts"))
   (gr_arc (start 83.560123 77.1) (mid 83.26723 77.807107) (end 82.560123 78.1)
@@
   (gr_line (start 83.560123 74.321277) (end 83.560123 77.1)
     (stroke (width 0.1) (type default)) (layer "Edge.Cuts"))
-  (gr_text "https://t.me/zx_delta_s" (at 106.0704 39.2176) (layer "B.SilkS")
+  (gr_text "https://t.me/zx_delta_s" (at 102.616 51.816 90) (layer "B.SilkS")
     (effects (font (size 0.75 0.75) (thickness 0.09375)) (justify left bottom mirror))
   )
@@
     (effects (font (size 1.5 1.5) (thickness 0.3) bold) (justify mirror))
   )
-  (gr_text "https://t.me/zx_delta_s" (at 77.6224 39.1922) (layer "B.SilkS")
+  (gr_text "https://t.me/zx_delta_s" (at 74.93 51.816 90) (layer "B.SilkS")
     (effects (font (size 0.75 0.75) (thickness 0.09375)) (justify left bottom mirror))
   )
@@
     (effects (font (size 1.5 1.5) (thickness 0.3) bold))
   )
-  (gr_text "MadCat 2023 Ver.1" (at 65.8368 38.4302) (layer "F.SilkS")
+  (gr_text "MadCat 2023 Ver.1" (at 72.39 76.454) (layer "F.SilkS")
     (effects (font (size 0.75 0.75) (thickness 0.09375)) (justify left top))
   )
@@
     (effects (font (size 0.75 0.75) (thickness 0.09375)) (justify left top))
   )
-  (gr_text "MadCat 2023 Ver.1" (at 93.8276 38.4556) (layer "F.SilkS")
+  (gr_text "MadCat 2023 Ver.1" (at 99.822 76.2) (layer "F.SilkS")
     (effects (font (size 0.75 0.75) (thickness 0.09375)) (justify left top))
   )
@@
     )
   )
+  (group "" (id cf7c8a5f-1386-4e15-864c-c49457855ac5)
+    (members
+      07d7d64b-4301-4964-899c-3b7c45dbb0b8
+      21e44455-29d0-4be7-9ffc-9f345782fbf1
+      2368b186-d9f8-4d23-aeca-24d52b47466a
+      4ca40101-d0d8-4a0b-9c14-c97a067eb962
+      4ece095c-1f35-48c3-b330-4e517277a006
+      b2bb3eb3-7876-4425-bf0d-823431ede5bb
+    )
+  )
